File: Ben6502.sch (KiCad schematic (older format))
At the start: 21 parts, among them SW1 1, SW2 1, SW3 1, SW4 1, SW5 1, U1 LCD-016M002B, U2 KM62256CLP, U3 W65C02S, U4 WD65C22, U5 8C256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

Commit message: finish first pass
Parts:
- added C2, C3, C4, C5: 100nf, Capacitor_THT:C_Rect_L4.6mm_W2.0mm_P2.50mm_MKS02_FKP02, symbol Device:C
- added H1, H2, H3, H4: MountingHole, MountingHole:MountingHole_2.5mm, symbol Mechanical:MountingHole
- added J1: DATA, Connector_PinSocket_2.54mm:PinSocket_1x08_P2.54mm_Vertical, symbol Connector:Conn_01x08_Female
- added J2: ADDR, Connector_PinSocket_2.54mm:PinSocket_1x16_P2.54mm_Vertical, symbol Connector:Conn_01x16_Female
- added J3: PWR, Connector_BarrelJack:BarrelJack_CUI_PJ-063AH_Horizontal_CircularHoles, symbol Connector:Barrel_Jack
- added RV1: 10k, Connector_PinHeader_2.54mm:PinHeader_1x03_P2.54mm_Vertical, symbol Device:R_POT
- C1: footprint (none) -> Capacitor_THT:C_Rect_L4.6mm_W2.0mm_P2.50mm_MKS02_FKP02
- R1, R2, R3, R4, R5, R6, R7: footprint (none) -> Resistor_THT:R_Axial_DIN0204_L3.6mm_D1.6mm_P7.62mm_Horizontal
- RESET1, SW1, SW2, SW3, SW4, SW5: footprint (none) -> Connector_PinHeader_2.54mm:PinHeader_1x02_P2.54mm_Vertical
- U2, U5: footprint (none) -> Package_DIP:DIP-28_W15.24mm_Socket_LongPads
- U3: footprint (none) -> Package_DIP:DIP-40_W15.24mm_Socket_LongPads
- U4: footprint Package_DIP:SMDIP-40_W15.24mm -> Package_DIP:DIP-40_W15.24mm_Socket_LongPads
- U6: footprint (none) -> Package_DIP:DIP-14_W7.62mm_Socket_LongPads
Connections:
- net +5V: now also U2.28 (VCC), U6.14 (VCC), C2.1, C3.1, C4.1, C5.1, J3.2
- net A0: now also J2.1 (Pin_1)
- net A1: now also J2.2 (Pin_2)
- net A10: now also J2.11 (Pin_11)
- net A11: now also J2.12 (Pin_12)
- net A12: now also J2.13 (Pin_13)
- net A13: now also J2.14 (Pin_14)
- net A14: now also J2.15 (Pin_15)
- net A15: now also J2.16 (Pin_16)
- net A2: now also J2.3 (Pin_3)
- net A3: now also J2.4 (Pin_4)
- net A4: now also J2.5 (Pin_5)
- net A5: now also J2.6 (Pin_6)
- net A6: now also J2.7 (Pin_7)
- net A7: now also J2.8 (Pin_8)
- net A8: now also J2.9 (Pin_9)
- net A9: now also J2.10 (Pin_10)
- net D0: now also J1.1 (Pin_1)
- net D1: now also J1.2 (Pin_2)
- net D2: now also J1.3 (Pin_3)
- net D3: now also J1.4 (Pin_4)
- net D4: now also J1.5 (Pin_5)
- net D5: now also J1.6 (Pin_6)
- net D6: now also J1.7 (Pin_7)
- net D7: now also J1.8 (Pin_8)
- net GND: now also U6.7 (GND), C2.2, C3.2, C4.2, C5.2, J3.1, RV1.1
- net at U1.3 (VO): now also RV1.2
- no-connect marks 11 -> 12
Other:
- moved on the sheet: C1, R1, R2, R3, R4, R5, R6, R7, RESET1, SW1, SW2, SW3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
